File: Shifter_demo/Shifter_demo.kicad_pcb (KiCad board)
At the start: 2 copper layers, 78 x 58 mm, 42 parts, among them J1 RST, J2 BSEL, J3 S06B-XASK-1, J4 SO4B-XASK-1, J5 S03B-XASK-1, J6 S03B-XASK-1, Q1 BSS205N, U1 ESP32-S3-WROOM-1U-N4R2, U2 LMR50410Y3FQDBVRQ1, U3 MAX3390EEUD_T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

Commit message: Add SCS checks to Schematic and PCB
Parts:
- added J7: S03B-XASK-1, Connector_JST:JST_XA_S03B-XASK-1_1x03_P2.50mm_Horizontal, F.Cu at (128.5, 118.0)
- added R12: 10k, Resistor_SMD:R_0805_2012Metric_Pad1.20x1.40mm_HandSolder, B.Cu at (106.5, 137.5)
- added R14: 10k, Resistor_SMD:R_0805_2012Metric_Pad1.20x1.40mm_HandSolder, B.Cu at (80.2, 135.5)
- added R15: 10k, Resistor_SMD:R_0805_2012Metric_Pad1.20x1.40mm_HandSolder, B.Cu at (80.2, 139.5)
- added R16: 10k, Resistor_SMD:R_0805_2012Metric_Pad1.20x1.40mm_HandSolder, B.Cu at (109.0, 137.5)
- added R17: 10k, Resistor_SMD:R_0805_2012Metric_Pad1.20x1.40mm_HandSolder, B.Cu at (82.2, 135.5)
- added R18: 10k, Resistor_SMD:R_0805_2012Metric_Pad1.20x1.40mm_HandSolder, B.Cu at (78.2, 135.5)
- added R19: 10k, Resistor_SMD:R_0805_2012Metric_Pad1.20x1.40mm_HandSolder, B.Cu at (78.2, 139.5)
- added R20: 10k, Resistor_SMD:R_0805_2012Metric_Pad1.20x1.40mm_HandSolder, B.Cu at (82.2, 139.5)
- added R21: 180, Resistor_SMD:R_0805_2012Metric_Pad1.20x1.40mm_HandSolder, B.Cu at (106.5, 133.5)
- added R22: 180, Resistor_SMD:R_0805_2012Metric_Pad1.20x1.40mm_HandSolder, B.Cu at (109.0, 133.5)
- added R23: 180, Resistor_SMD:R_0805_2012Metric_Pad1.20x1.40mm_HandSolder, B.Cu at (104.0, 133.5)
- added R24: 5k8, Resistor_SMD:R_0805_2012Metric_Pad1.20x1.40mm_HandSolder, B.Cu at (104.5, 141.0)
- added R25: 10k, Resistor_SMD:R_0805_2012Metric_Pad1.20x1.40mm_HandSolder, B.Cu at (108.5, 141.0)
- added R26: 12k, Resistor_SMD:R_0805_2012Metric_Pad1.20x1.40mm_HandSolder, B.Cu at (104.5, 143.5)
- added R27: 10k, Resistor_SMD:R_0805_2012Metric_Pad1.20x1.40mm_HandSolder, B.Cu at (108.5, 143.5)
- added R8: 10k, Resistor_SMD:R_0805_2012Metric_Pad1.20x1.40mm_HandSolder, B.Cu at (104.0, 137.5)
- added U5: LM339, CustomFootprints:LM339DR, B.Cu at (96.3, 138.0)
- added U6: LM339, CustomFootprints:LM339DR, B.Cu at (87.2, 138.0)
- added U8: CD4081, CustomFootprints:D14, B.Cu at (72.2, 138.2)
- J3: value S06B-XASK-1 -> S03B-XASK-1; footprint Connector_JST:JST_XA_S06B-XASK-1_1x06_P2.50mm_Horizontal -> Connector_JST:JST_XA_S03B-XASK-1_1x03_P2.50mm_Horizontal
- J6: value S03B-XASK-1 -> SO4B-XASK-1; footprint Connector_JST:JST_XA_S03B-XASK-1_1x03_P2.50mm_Horizontal -> Connector_JST:JST_XA_S04B-XASK-1_1x04_P2.50mm_Horizontal
- moved J3 9.00 mm to (128.5, 106.0)
- moved J4 3.30 mm to (128.5, 133.2)
- moved J6 2.65 mm to (113.0, 136.0)
- moved REF** 0.79 mm to (86.8, 116.8)
Connections:
- J3 pad 1: GND -> E_MOSI
- J3 pad 2: E_CS -> E_MISO
- J3 pad 3: E_SCLK -> +5V
- J4 pad 1: NEUTRAL -> SHIFT_NEUTRAL
- J4 pad 4: ECU -> +3V3
- U1 pad : GND -> (no net)
- U1 pad 24: unconnected-(U1-IO47-Pad24) -> UP
- U1 pad 25: unconnected-(U1-IO48-Pad25) -> DOWN
- U1 pad 26: unconnected-(U1-IO45-Pad26) -> NEUTRAL
Routing:
- net +3V3: track 102.4 -> 197.8 mm, vias 1 -> 6
- net +5V: track 154.9 -> 243.2 mm, vias 1 -> 4
- net Net-(R19-Pad2): track 0.00 -> 34.1 mm
- net Net-(R20-Pad2): track 0.00 -> 31.5 mm, vias 0 -> 2
- net Net-(U6A--): track 0.00 -> 27.8 mm, vias 0 -> 2
- net ECU: track 9.94 -> 37.2 mm, vias 0 -> 2
- net Net-(R15-Pad2): track 0.00 -> 27.3 mm
- net Net-(R18-Pad1): track 0.00 -> 27.0 mm, vias 0 -> 2
- net SHIFT_UP: track 0.00 -> 26.3 mm
- net Net-(R17-Pad1): track 0.00 -> 25.2 mm, vias 0 -> 2
- net NEUTRAL: track 0.00 -> 25.2 mm, vias 0 -> 2
- net DOWN: track 0.00 -> 23.7 mm, vias 0 -> 2
- net Net-(R14-Pad1): track 0.00 -> 23.5 mm, vias 0 -> 3
- net SHIFT_DOWN: track 0.00 -> 22.7 mm
- net 3.5V Ref: track 0.00 -> 20.0 mm
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