File: hardware/Shifter.kicad_sch (KiCad schematic)
At the start: 62 parts, among them J1 RST, J2 BSEL, J3 S03B-XASK-1, J4 SO4B-XASK-1, J5 S03B-XASK-1, J6 SO4B-XASK-1, J7 S03B-XASK-1, J8 SO4B-XASK-1, J9 Conn_01x02, Q1 BSS205N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

Commit message: ready to go
Parts:
- removed R12, R16, R8: 10k, Resistor_SMD:R_0603_1608Metric, symbol Device:R
- removed R21, R22, R23: 180, Resistor_SMD:R_0603_1608Metric, symbol Device:R
- U5, U6: value LM339 -> TLV1704; footprint CustomFootprints:LM339DR -> CustomFootprints:PW14_TEX
Connections:
- net SHIFT_DOWN: now also TP2.1, U5.10 (-), U5.9 (+)
- net SHIFT_NEUTRAL: now also TP10.1, U6.4 (-), U6.7 (+)
- net SHIFT_UP: now also TP4.1, U5.4 (-), U5.7 (+)
