File: hardware/Shifter.kicad_sch (KiCad schematic)
At the start: 56 parts, among them J1 RST, J2 BSEL, J3 S03B-XASK-1, J4 SO4B-XASK-1, J5 S03B-XASK-1, J6 SO4B-XASK-1, J7 S03B-XASK-1, J8 SO4B-XASK-1, J9 Conn_01x02, Q1 BSS205N, U1 ESP32-S3-WROOM-1U-N4R2, U2 LMR50410Y3FQDBVRQ1, U3 MAX3390EEUD_T, U4 ISO1042BQDWVQ1, U5 TLV1704, U6 TLV1704

Commit message: minor changes
Other:
- company: (none) -> Manchester Stinger Motorsports
- title: (none) -> Gear-shifter
