File: hardware/Shifter.kicad_pcb (KiCad board)
At the start: 4 copper layers, 78 x 58 mm, 59 parts, among them J1 RST, J2 BSEL, J3 S03B-XASK-1, J4 SO4B-XASK-1, J5 S03B-XASK-1, J6 SO4B-XASK-1, J7 S03B-XASK-1, J8 SO4B-XASK-1, J9 Conn_01x02, Q1 BSS205N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

Commit message: rob-proofing
Parts:
- removed the G*** at (90.9, 117.2)
- removed the REF** at (185.0, 117.0)
- added G***: LOGO, LOGO, F.Cu at (91.5, 117.0)
Routing:
- net +5V: track 219.2 -> 225.5 mm
Other:
- board text added: "Designed by James Platt Manchester Stinger Motorsports 2026 Thanks to: Robertas Barkauskas Mark Matvijcsuk Shreyas Vartia"
- board text removed: "Designed by James Platt Manchester Stinger Motorsports 2025 Thanks to: Robertas Barkauskas Mark Matvijcsuk Shreyas Vartia"
- board text removed: "Powered by"

Commit message: ready to go
Parts:
- C2: value 22u -> 10u
- R24: value 5k8 -> 5k6
- U5, U6: value LM339 -> TLV1704; footprint CustomFootprints:LM339DR -> CustomFootprints:PW14_TEX
- moved U6 2.55 mm to (84.8, 137.5)
- moved U5 1.61 mm to (94.8, 137.5)
Connections:
- U5 pad 10: Net-(U5C--) -> SHIFT_DOWN
- U5 pad 4: Net-(U5A--) -> SHIFT_UP
- U5 pad 7: Net-(U5A--) -> SHIFT_UP
- U5 pad 9: Net-(U5C--) -> SHIFT_DOWN
- U6 pad 4: Net-(U6A--) -> SHIFT_NEUTRAL
- U6 pad 7: Net-(U6A--) -> SHIFT_NEUTRAL
Routing:
- net SHIFT_NEUTRAL: track 20.9 -> 51.5 mm, vias 0 -> 2
- net Net-(U6A--): track 27.8 -> 2.00 mm, vias 2 -> 1
- net SHIFT_DOWN: track 23.7 -> 42.4 mm, vias 0 -> 2
- net Net-(U5A--): track 18.5 -> 2.00 mm, vias 2 -> 0
- net SHIFT_UP: track 27.3 -> 38.7 mm
- net Net-(U5C--): track 17.3 -> 8.16 mm, vias 2 -> 1
- net +5V: track 225.5 -> 232.2 mm, vias 3 -> 6
- net 2.5V Ref: track 19.8 -> 24.1 mm
- net 3.5V Ref: track 20.0 -> 23.7 mm, vias 0 -> 2
- net GND: track 12.2 -> 15.4 mm
- net NEUTRAL: track 21.0 -> 18.9 mm
- net UP: track 24.0 -> 22.6 mm
- net DOWN: track 21.5 -> 20.4 mm

Commit message: actually good to go
Routing:
- net Net-(U5C--): track 8.16 -> 6.35 mm, vias 1 -> 0
- net Net-(U6A--): vias 1 -> 0
